File: pmtcmini-h10721/pmtcmini-h10721.kicad_pcb (KiCad board)
At the start: 2 copper layers, 19.5 x 39.1 mm, 29 parts, among them J1 Conn_01x03, J2 Conn_01x05, P1 ZX62M-B-5P(01), U1 MAX6106EUR-T, U2 MAX5214GUAT, U3 STM32F042F6P6, U4 ADP7118AUJZ-3.3-R7, U5 TPS22918TDBVTQ1, U6 ADP7118AUJZ-3.3-R7

Commit message: revB sch & pcb
Parts:
- removed P1: ZX62M-B-5P(01), HRS_ZX62M-B-5P(01)
- added J3: 10104110-0001LF, 10104110-0001LF, F.Cu at (136.5, 53.8)
- added R8: 49.9, Resistor_SMD:R_0402_1005Metric, F.Cu at (133.5, 87.0)
Connections:
- C1 pad 2: GNDA -> GND
- C11 pad 1: /PMT_ADJ -> Net-(C11-Pad1)
- C6 pad 2: GNDA -> GND
- C8 pad 2: GNDA -> GND
- J1 pad 2: /PMT_ADJ -> Net-(C11-Pad1)
- U1 pad 3: GNDA -> GND
- U2 pad 8: GNDA -> GND
Routing:
- net GNDA: track 9.74 -> 0.00 mm, vias 3 -> 0
- net GND: track 20.8 -> 29.5 mm, vias 11 -> 14
- net VBUS: track 50.8 -> 58.2 mm
- net /PMT_ADJ: track 9.16 -> 2.70 mm
- net Net-(C11-Pad1): track 0.00 -> 5.73 mm
- net +3V3: track 22.7 -> 17.6 mm, vias 8 -> 4
- net (no net): vias 0 -> 4
- removed copper zone on B.Cu, net GNDA
Other:
- board text added: "PMTCMini-H10721 Rev B Eben Olson 2018"
- board text removed: "PMTCMini-H10721 Rev A Eben Olson 2018"
