File: kicad/pmtcmini-h10770.sch (KiCad schematic (older format))
At the start: 30 parts, among them J1 Conn_01x03, J2 Conn_01x05, J3 10104110-0001LF, U1 MAX6106EUR-T, U2 MAX5214GUAT, U3 STM32F042F6P6, U4 ADP7118AUJZ-3.3-R7, U5 TPS22918TDBVTQ1, U6 ADP7118AUJZ-3.3-R7

Commit message: h10770 revA
Parts:
- added J4: DROK_Voltage_Converter, symbol DROK-Voltage_Converter:DROK_Voltage_Converter
- added R10, R9: 500, Resistor_SMD:R_0402_1005Metric, symbol Device:R
- added R11: 1.5k, Resistor_SMD:R_0402_1005Metric, symbol Device:R
- U5: value TPS22918TDBVTQ1 -> TPS22810-Q1; symbol TPS22918TDBVTQ1:TPS22918TDBVTQ1 -> TPS22810-Q1:TPS22810-Q1; Arrow Part Number TPS22918TDBVTQ1 -> TPS22810-Q1; Description TEXAS INSTRUMENTS - TPS22918TDBVTQ1 - POWER LOAD SWITCH, AE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 -> (none); Manufacturer_Part_Number TPS22918TDBVTQ1 -> TPS22810-Q1
Connections:
- net labels added: V+
- wire segments 91 -> 104
Changed lines of the file:
@@
 EESchema Schematic File Version 4
-LIBS:pmtcmini-h10721-cache
+LIBS:pmtcmini-h10770-cache
 EELAYER 26 0
 EELAYER END
@@
 L Connector_Generic:Conn_01x05 J2
 U 1 1 5B2BD838
-P 10100 4250
-F 0 "J2" H 10180 4292 50  0000 L CNN
-F 1 "Conn_01x05" H 10180 4201 50  0000 L CNN
-F 2 "Connector_Molex:Molex_PicoBlade_53047-1010_1x05_P1.25mm_Vertical" H 10100 4250 50  0001 C CNN
-F 3 "~" H 10100 4250 50  0001 C CNN
-	1    10100 4250
+P 10300 3900
+F 0 "J2" H 10380 3942 50  0000 L CNN
+F 1 "Conn_01x05" H 10380 3851 50  0000 L CNN
+F 2 "Connector_Molex:Molex_PicoBlade_53047-1010_1x05_P1.25mm_Vertical" H 10300 3900 50  0001 C CNN
+F 3 "~" H 10300 3900 50  0001 C CNN
+	1    10300 3900
 	1    0    0    -1
 $EndComp
@@
 L power:+3.3V #PWR025
 U 1 1 5B2BE943
-P 9750 4050
-F 0 "#PWR025" H 9750 3900 50  0001 C CNN
-F 1 "+3.3V" H 9765 4223 50  0000 C CNN
-F 2 "" H 9750 4050 50  0001 C CNN
-F 3 "" H 9750 4050 50  0001 C CNN
-	1    9750 4050
-	1    0    0    -1
-$EndComp
-Wire Wire Line
-	9900 4050 9750 4050
-Wire Wire Line
-	9900 4150 9500 4150
-Wire Wire Line
-	9900 4250 9500 4250
-Wire Wire Line
-	9900 4350 9500 4350
+P 9950 3700
+F 0 "#PWR025" H 9950 3550 50  0001 C CNN
+F 1 "+3.3V" H 9965 3873 50  0000 C CNN
+F 2 "" H 9950 3700 50  0001 C CNN
+F 3 "" H 9950 3700 50  0001 C CNN
+	1    9950 3700
+	1    0    0    -1
+$EndComp
+Wire Wire Line
+	10100 3700 9950 3700
+Wire Wire Line
+	10100 3800 9700 3800
+Wire Wire Line
+	10100 3900 9700 3900
+Wire Wire Line
+	10100 4000 9700 4000
 $Comp
 L power:GND #PWR026
 U 1 1 5B2BED43
-P 9750 4450
-F 0 "#PWR026" H 9750 4200 50  0001 C CNN
-F 1 "GND" H 9755 4277 50  0000 C CNN
-F 2 "" H 9750 4450 50  0001 C CNN
-F 3 "" H 9750 4450 50  0001 C CNN
-	1    9750 4450
-	1    0    0    -1
-$EndComp
-Wire Wire Line
-	9750 4450 9900 4450
-Text Label 9500 4150 0    50   ~ 0
+P 9950 4100
+F 0 "#PWR026" H 9950 3850 50  0001 C CNN
+F 1 "GND" H 9955 3927 50  0000 C CNN
+F 2 "" H 9950 4100 50  0001 C CNN
+F 3 "" H 9950 4100 50  0001 C CNN
+	1    9950 4100
+	1    0    0    -1
+$EndComp
+Wire Wire Line
+	9950 4100 10100 4100
+Text Label 9700 3800 0    50   ~ 0
 SWDIO
-Text Label 9500 4250 0    50   ~ 0
+Text Label 9700 3900 0    50   ~ 0
 SWCLK
-Text Label 9500 4350 0    50   ~ 0
+Text Label 9700 4000 0    50   ~ 0
 RESET
 Wire Wire Line
@@
 	0    -1   -1   0
 $EndComp
-$Comp
-L power:+3.3V #PWR019
-U 1 1 5B31FA47
-P 6350 4550
-F 0 "#PWR019" H 6350 4400 50  0001 C CNN
-F 1 "+3.3V" H 6365 4723 50  0000 C CNN
-F 2 "" H 6350 4550 50  0001 C CNN
-F 3 "" H 6350 4550 50  0001 C CNN
-	1    6350 4550
-	1    0    0    -1
-$EndComp
-Wire Wire Line
-	6350 4550 6350 4650
 Wire Wire Line
 	6350 4850 6000 4850
@@
 PMT_VDD
 $Comp
-L TPS22918TDBVTQ1:TPS22918TDBVTQ1 U5
+L TPS22810-Q1:TPS22810-Q1 U5
 U 1 1 5B33C77A
 P 6350 4650
 F 0 "U5" H 6900 4915 50  0000 C CNN
-F 1 "TPS22918TDBVTQ1" H 6900 4824 50  0000 C CNN
+F 1 "TPS22810-Q1" H 6900 4824 50  0000 C CNN
 F 2 "SOT95P280X100-6N" H 7300 4750 50  0001 L CNN
-F 3 "http://www.ti.com/general/docs/lit/getliterature.tsp?genericPartNumber=TPS22918-Q1&fileType=pdf" H 7300 4650 50  0001 L CNN
-F 4 "TEXAS INSTRUMENTS - TPS22918TDBVTQ1 - POWER LOAD SWITCH, AEC-Q100, 5.5V, SOT23" H 7300 4550 50  0001 L CNN "Description"
-F 5 "1" H 7300 4450 50  0001 L CNN "Height"
-F 6 "Texas Instruments" H 7300 4350 50  0001 L CNN "Manufacturer_Name"
-F 7 "TPS22918TDBVTQ1" H 7300 4250 50  0001 L CNN "Manufacturer_Part_Number"
-F 8 "" H 7300 4150 50  0001 L CNN "RS Part Number"
-F 9 "" H 7300 4050 50  0001 L CNN "RS Price/Stock"
-F 10 "TPS22918TDBVTQ1" H 7300 3950 50  0001 L CNN "Arrow Part Number"
-F 11 "" H 7300 3850 50  0001 L CNN "Arrow Price/Stock"
+F 3 "" H 7300 4650 50  0001 L CNN
+F 4 "1" H 7300 4450 50  0001 L CNN "Height"
+F 5 "Texas Instruments" H 7300 4350 50  0001 L CNN "Manufacturer_Name"
+F 6 "TPS22810-Q1" H 7300 4250 50  0001 L CNN "Manufacturer_Part_Number"
+F 7 "TPS22810-Q1" H 7300 3950 50  0001 L CNN "Arrow Part Number"
 	1    6350 4650
 	1    0    0    -1
@@
 L power:GNDA #PWR0105
 U 1 1 5B3FA3AB
-P 10000 5550
-F 0 "#PWR0105" H 10000 5300 50  0001 C CNN
-F 1 "GNDA" H 10005 5377 50  0000 C CNN
-F 2 "" H 10000 5550 50  0001 C CNN
-F 3 "" H 10000 5550 50  0001 C CNN
-	1    10000 5550
+P 10450 6150
+F 0 "#PWR0105" H 10450 5900 50  0001 C CNN
+F 1 "GNDA" H 10455 5977 50  0000 C CNN
+F 2 "" H 10450 6150 50  0001 C CNN
+F 3 "" H 10450 6150 50  0001 C CNN
+	1    10450 6150
 	1    0    0    -1
 $EndComp
@@
 L power:GND #PWR0106
 U 1 1 5B3FA3B1
-P 9700 5550
-F 0 "#PWR0106" H 9700 5300 50  0001 C CNN
-F 1 "GND" H 9705 5377 50  0000 C CNN
-F 2 "" H 9700 5550 50  0001 C CNN
-F 3 "" H 9700 5550 50  0001 C CNN
-	1    9700 5550
-	1    0    0    -1
-$EndComp
-Wire Wire Line
-	9700 5550 10000 5550
+P 10150 6150
+F 0 "#PWR0106" H 10150 5900 50  0001 C CNN
+F 1 "GND" H 10155 5977 50  0000 C CNN
+F 2 "" H 10150 6150 50  0001 C CNN
+F 3 "" H 10150 6150 50  0001 C CNN
+	1    10150 6150
+	1    0    0    -1
+$EndComp
+Wire Wire Line
+	10150 6150 10450 6150
 $Comp
 L Device:R R8
@@
 	1    0    0    -1
 $EndComp
+$Comp
+L DROK-Voltage_Converter:DROK_Voltage_Converter J4
+U 1 1 5B40BC31
+P 10050 5000
+F 0 "J4" H 10129 5000 50  0000 L CNN
+F 1 "DROK_Voltage_Converter" H 10129 4909 50  0000 L CNN
+F 2 "" H 10050 5000 50  0001 C CNN
+F 3 "~" H 10050 5000 50  0001 C CNN
+	1    10050 5000
+	1    0    0    -1
+$EndComp
+$Comp
+L power:VBUS #PWR016
+U 1 1 5B412085
+P 9750 4800
+F 0 "#PWR016" H 9750 4650 50  0001 C CNN
+F 1 "VBUS" H 9765 4973 50  0000 C CNN
+F 2 "" H 9750 4800 50  0001 C CNN
+F 3 "" H 9750 4800 50  0001 C CNN
+	1    9750 4800
+	1    0    0    -1
+$EndComp
+Wire Wire Line
+	9750 4800 9850 4800
+$Comp
+L power:GND #PWR07
+U 1 1 5B4151C5
+P 8850 5550
+F 0 "#PWR07" H 8850 5300 50  0001 C CNN
+F 1 "GND" H 8855 5377 50  0000 C CNN
+F 2 "" H 8850 5550 50  0001 C CNN
+F 3 "" H 8850 5550 50  0001 C CNN
+	1    8850 5550
+	1    0    0    -1
+$EndComp
+Wire Wire Line
+	9400 5100 9850 5100
+Wire Wire Line
+	9850 4900 9400 4900
+Wire Wire Line
+	9400 4900 9400 5100
+$Comp
+L Device:R R11
+U 1 1 5B421F00
+P 9700 5300
+F 0 "R11" H 9630 5254 50  0000 R CNN
+F 1 "1.5k" H 9630 5345 50  0000 R CNN
+F 2 "Resistor_SMD:R_0402_1005Metric" V 9630 5300 50  0001 C CNN
+F 3 "~" H 9700 5300 50  0001 C CNN
+	1    9700 5300
+	0    -1   -1   0
+$EndComp
+Wire Wire Line
+	9850 5200 8850 5200
+Wire Wire Line
+	8850 5200 8850 5250
+$Comp
+L Device:R R10
+U 1 1 5B435585
+P 8850 5400
+F 0 "R10" H 8780 5354 50  0000 R CNN
+F 1 "500" H 8780 5445 50  0000 R CNN
+F 2 "Resistor_SMD:R_0402_1005Metric" V 8780 5400 50  0001 C CNN
+F 3 "~" H 8850 5400 50  0001 C CNN
+	1    8850 5400
+	-1   0    0    1
+$EndComp
+$Comp
+L Device:R R9
+U 1 1 5B438B42
+P 8550 5150
+F 0 "R9" H 8480 5104 50  0000 R CNN
+F 1 "500" H 8480 5195 50  0000 R CNN
+F 2 "Resistor_SMD:R_0402_1005Metric" V 8480 5150 50  0001 C CNN
+F 3 "~" H 8550 5150 50  0001 C CNN
+	1    8550 5150
+	-1   0    0    1
+$EndComp
+Wire Wire Line
+	9850 5000 8550 5000
+Wire Wire Line
+	8550 5300 8550 5550
+Wire Wire Line
+	8550 5550 8850 5550
+Connection ~ 8850 5550
+Wire Wire Line
+	9400 5100 9400 5550
+Wire Wire Line
+	9400 5550 8850 5550
+Connection ~ 9400 5100
+Wire Wire Line
+	9550 5300 9550 4800
+Wire Wire Line
+	9550 4800 9750 4800
+Connection ~ 9750 4800
+Text Label 9700 5000 0    50   ~ 0
+V+
+Text Label 6100 4650 0    50   ~ 0
+V+
+Wire Wire Line
+	6100 4650 6350 4650
 $EndSCHEMATC

Commit message: cleanup
Parts:
- J4: footprint (none) -> libraries:DROK_Voltage_Converter
Changed lines of the file:
@@
 F 0 "J4" H 10129 5000 50  0000 L CNN
 F 1 "DROK_Voltage_Converter" H 10129 4909 50  0000 L CNN
-F 2 "" H 10050 5000 50  0001 C CNN
+F 2 "libraries:DROK_Voltage_Converter" H 10050 5000 50  0001 C CNN
 F 3 "~" H 10050 5000 50  0001 C CNN
 	1    10050 5000
