File: kicad/pmtcmini-h10770.sch (KiCad schematic (older format))
At the start: 23 parts, among them IC1 STM32F042G6U6, J1 Conn_01x04, J2 Conn_01x05, J3 10118194-0001LF, J4 DROK_Voltage_Converter, U1 MAX6106EUR-T, U2 MAX5214GUAT, U4 ADP7118AUJZ-3.3-R7, U5 TPS22810-Q1, U6 ADP7118AUJZ-3.3-R7

Commit message: revB
Parts:
- removed D1: LED, LED_SMD:LED_0603_1608Metric, symbol Device:LED_Small
- removed R3: 1.5k, libraries:R_0603_1608Metric, symbol Device:R_Small_US
- J1: footprint libraries:PinHeader_1x04_P2.54mm_Vertical -> libraries:PinHeader_1x03_P2.54mm_Vertical; symbol Connector_Generic:Conn_01x04 -> Connector_Generic:Conn_01x03
Connections:
- net LED: no longer names the net of IC1.15 (PB1)
- no-connect marks 3 -> 2
Changed lines of the file:
@@
 EESchema Schematic File Version 4
 LIBS:pmtcmini-h10770-cache
-EELAYER 30 0
+EELAYER 29 0
 EELAYER END
 $Descr A4 11693 8268
@@
 $EndDescr
 $Comp
-L Connector_Generic:Conn_01x04 J1
+L Connector_Generic:Conn_01x03 J1
 U 1 1 5B2BD72A
 P 10100 2650
 F 0 "J1" H 10019 2325 50  0000 C CNN
 F 1 "Conn_01x04" H 10450 2450 50  0000 C CNN
-F 2 "libraries:PinHeader_1x04_P2.54mm_Vertical" H 10100 2650 50  0001 C CNN
+F 2 "libraries:PinHeader_1x03_P2.54mm_Vertical" H 10100 2650 50  0001 C CNN
 F 3 "~" H 10100 2650 50  0001 C CNN
 	1    10100 2650
@@
 $EndComp
 $Comp
-L Device:LED_Small D1
-U 1 1 5B2BE2AD
-P 3950 2200
-F 0 "D1" V 3988 2083 50  0000 R CNN
-F 1 "LED" V 3897 2083 50  0000 R CNN
-F 2 "LED_SMD:LED_0603_1608Metric" H 3950 2200 50  0001 C CNN
-F 3 "~" H 3950 2200 50  0001 C CNN
-	1    3950 2200
-	0    -1   -1   0
-$EndComp
-$Comp
 L power:GND #PWR028
 U 1 1 5B2BE3DD
@@
 	1    0    0    -1
 $EndComp
-$Comp
-L Device:R_Small_US R3
-U 1 1 5B2D41E2
-P 3950 1900
-F 0 "R3" H 4020 1946 50  0000 L CNN
-F 1 "1.5k" H 4020 1855 50  0000 L CNN
-F 2 "libraries:R_0603_1608Metric" V 3880 1900 50  0001 C CNN
-F 3 "~" H 3950 1900 50  0001 C CNN
-	1    3950 1900
-	1    0    0    -1
-$EndComp
-$Comp
-L power:+3.3V #PWR010
-U 1 1 5B2D43E9
-P 3950 1750
-F 0 "#PWR010" H 3950 1600 50  0001 C CNN
-F 1 "+3.3V" H 3965 1923 50  0000 C CNN
-F 2 "" H 3950 1750 50  0001 C CNN
-F 3 "" H 3950 1750 50  0001 C CNN
-	1    3950 1750
-	1    0    0    -1
-$EndComp
-Text Label 3400 2500 0    50   ~ 0
-LED
 Text Label 3750 2150 2    50   ~ 0
 USBP
@@
 	1150 2900 1550 2900
 Wire Wire Line
-	3350 2500 3950 2500
-Wire Wire Line
 	6450 1200 6450 1100
 Wire Wire Line
@@
 	0    -1   -1   0
 $EndComp
-Wire Wire Line
-	3950 1800 3950 1750
-Wire Wire Line
-	3950 2100 3950 2000
-Wire Wire Line
-	3950 2300 3950 2500
 Text Label 9600 5200 0    50   ~ 0
 -12V
@@
 	7900 1000 7900 1200
 Connection ~ 7900 1200
-NoConn ~ 9900 2450
 $EndSCHEMATC

Commit message: revC, bugfixes
Parts:
- J2: symbol Connector_Generic:Conn_01x06 -> Connector_Generic:Conn_01x04
- R10, R9: footprint libraries:R_0805_2012Metric -> libraries:R_1206_3216Metric
Connections:
- net +3V3: now also IC1.18 (VDDIO2); no longer J2.1 (Pin_1)
- net GND: now also J2.4 (Pin_4); no longer J2.6 (Pin_6)
- net MOSI: now also IC1.10 (PA4); no longer IC1.13 (PA7)
- net RESET: now also J2.3 (Pin_3); no longer J2.4 (Pin_4)
- net SWCLK: now also J2.2 (Pin_2); no longer J2.3 (Pin_3)
- net SWDIO: now also J2.1 (Pin_1); no longer J2.2 (Pin_2)
- net ~CS: now also IC1.13 (PA7); no longer IC1.10 (PA4)
- no-connect marks 2 -> 1
Changed lines of the file:
@@
 EESchema Schematic File Version 4
-LIBS:pmtcmini-h10770-cache
-EELAYER 29 0
+EELAYER 30 0
 EELAYER END
 $Descr A4 11693 8268
@@
 $EndComp
 $Comp
-L Connector_Generic:Conn_01x06 J2
+L Connector_Generic:Conn_01x04 J2
 U 1 1 5B2BD838
 P 10300 3900
@@
 Text Label 9650 1400 0    50   ~ 0
 USBM
-$Comp
-L power:+3.3V #PWR025
-U 1 1 5B2BE943
-P 9950 3650
-F 0 "#PWR025" H 9950 3500 50  0001 C CNN
-F 1 "+3.3V" H 9965 3823 50  0000 C CNN
-F 2 "" H 9950 3650 50  0001 C CNN
-F 3 "" H 9950 3650 50  0001 C CNN
-	1    9950 3650
-	1    0    0    -1
-$EndComp
-Wire Wire Line
-	10100 3700 9950 3700
 Wire Wire Line
 	10100 3800 9700 3800
@@
 L power:GND #PWR026
 U 1 1 5B2BED43
-P 9950 4250
-F 0 "#PWR026" H 9950 4000 50  0001 C CNN
-F 1 "GND" H 9955 4077 50  0000 C CNN
-F 2 "" H 9950 4250 50  0001 C CNN
-F 3 "" H 9950 4250 50  0001 C CNN
-	1    9950 4250
-	1    0    0    -1
-$EndComp
-Wire Wire Line
-	9950 4200 10100 4200
+P 9950 4150
+F 0 "#PWR026" H 9950 3900 50  0001 C CNN
+F 1 "GND" H 9955 3977 50  0000 C CNN
+F 2 "" H 9950 4150 50  0001 C CNN
+F 3 "" H 9950 4150 50  0001 C CNN
+	1    9950 4150
+	1    0    0    -1
+$EndComp
+Wire Wire Line
+	9950 4100 10100 4100
 Text Label 9700 3800 0    50   ~ 0
 SWDIO
@@
 Wire Wire Line
 	1150 2800 1550 2800
-Text Label 1150 2800 0    50   ~ 0
+Text Label 1150 3100 0    50   ~ 0
 ~CS
 Text Label 1150 2900 0    50   ~ 0
 SCLK
-Text Label 1150 3100 0    50   ~ 0
+Text Label 1150 2800 0    50   ~ 0
 MOSI
 Wire Wire Line
@@
 F 0 "R10" H 8780 5354 50  0000 R CNN
 F 1 "500" H 8780 5445 50  0000 R CNN
-F 2 "libraries:R_0805_2012Metric" V 8780 5400 50  0001 C CNN
+F 2 "libraries:R_1206_3216Metric" V 8780 5400 50  0001 C CNN
 F 3 "~" H 8850 5400 50  0001 C CNN
 	1    8850 5400
@@
 F 0 "R9" H 8480 5104 50  0000 R CNN
 F 1 "500" H 8480 5195 50  0000 R CNN
-F 2 "libraries:R_0805_2012Metric" V 8480 5150 50  0001 C CNN
+F 2 "libraries:R_1206_3216Metric" V 8480 5150 50  0001 C CNN
 F 3 "~" H 8550 5150 50  0001 C CNN
 	1    8550 5150
@@
 Wire Wire Line
 	7900 1250 7900 1200
-NoConn ~ 10100 4100
-Wire Wire Line
-	9950 3700 9950 3650
-Wire Wire Line
-	9950 4250 9950 4200
+Wire Wire Line
+	9950 4150 9950 4100
 Wire Wire Line
 	9750 4800 9750 4700
@@
 	7900 1000 7900 1200
 Connection ~ 7900 1200
+$Comp
+L power:+3.3V #PWR0108
+U 1 1 6014548A
+P 4025 2175
+F 0 "#PWR0108" H 4025 2025 50  0001 C CNN
+F 1 "+3.3V" V 4025 2325 50  0000 L CNN
+F 2 "" H 4025 2175 50  0001 C CNN
+F 3 "" H 4025 2175 50  0001 C CNN
+	1    4025 2175
+	1    0    0    -1
+$EndComp
+Wire Wire Line
+	3350 2350 4025 2350
+Wire Wire Line
+	4025 2175 4025 2350
 $EndSCHEMATC
